Commit message: Update tcp orientation to make z axis inward

File: demo/model/reach_study.xacro (robot description, xacro)
@@ -7,5 +7,5 @@
     <parent link="tool0"/>
     <child link="tcp"/>
-    <origin xyz="0 0 0.1" rpy="0 0 0"/>
+    <origin xyz="0 0 0.1" rpy="3.14 0 0"/>
   </joint>
 </robot>

Commit message: Use builtin function for 180 angle

File: demo/model/reach_study.xacro (robot description, xacro)
@@ -7,5 +7,5 @@
     <parent link="tool0"/>
     <child link="tcp"/>
-    <origin xyz="0 0 0.1" rpy="3.14 0 0"/>
+    <origin xyz="0 0 0.1" rpy="${radians(180)} 0 0"/>
   </joint>
 </robot>
